File: 3x4 keypad.kicad_sch (KiCad schematic)
At the start: 25 parts, among them J1 Conn_01x07_Pin, SW1 SW_Push, SW10 SW_Push, SW11 SW_Push, SW12 SW_Push, SW2 SW_Push, SW3 SW_Push, SW4 SW_Push, SW5 SW_Push, SW6 SW_Push, SW7 SW_Push, SW8 SW_Push, SW9 SW_Push

Commit message: some connectors changed and added footprints but pcb still needs work
Parts:
- removed J1: Conn_01x07_Pin, symbol Connector:Conn_01x07_Pin
- removed SW1, SW10, SW11, SW12, SW2, SW3, SW4, SW5, SW6, SW7, SW8, SW9: SW_Push, symbol Switch:SW_Push
- added J1: Conn_01x07_Pin, Connector_Hirose:Hirose_DF13-07P-1.25DS_1x07_P1.25mm_Horizontal, symbol custom:Conn_01x07_Pin
- added SW1, SW10, SW11, SW12, SW2, SW3, SW4, SW5, SW6, SW7, SW8, SW9: SW_Push, Button_Switch_THT:SW_CW_GPTS203211B, symbol custom:SW_Push
Connections:
- net at D5.1 (K): now also SW5.1
- net at D11.2 (A), D2.2 (A), D5.2 (A)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: now also J1.6 (Pin_6)
- net at D11.1 (K): now also SW11.1
- net at D1.2 (A), D12.2 (A), D6.2 (A)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: now also J1.5 (Pin_5)
- net at D10.2 (A), D3.2 (A), D4.2 (A)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: now also J1.7 (Pin_7)
- net at D1.1 (K): now also SW1.1
- net at D7.1 (K): now also SW7.1
- net at D6.1 (K): now also SW4.1
- net at D8.1 (K): now also SW8.1
- net at D12.1 (K): now also SW10.1
- net at D9.1 (K): now also SW9.1
- net at D4.1 (K): now also SW6.1
- net at D2.1 (K): now also SW2.1
- net at D10.1 (K): now also SW12.1
- net at D3.1 (K): now also SW3.1
- new net: J1.1 (Pin_1), SW1.2, SW2.2, SW3.2
- new net: J1.3 (Pin_3), SW7.2, SW8.2, SW9.2
- new net: J1.2 (Pin_2), SW4.2, SW5.2, SW6.2
- new net: J1.4 (Pin_4), SW10.2, SW11.2, SW12.2
